Commit message: new 6 robot

File: lab6/ex4_ex5/my_robot/robot_description/urdf/depth.urdf.xacro (robot description, xacro)
@@ -5,5 +5,5 @@
         <parent link="base_link"/>
         <child link="depth_frame"/>
-        <origin xyz="0.1 0 0.25" rpy="0 0 0"/>
+        <origin xyz="0.15 0.05 0.25" rpy="0 0 0"/>
     </joint>
     <material name="aluminum">

File: lab6/ex4_ex5/my_robot/robot_description/urdf/gazebo.urdf.xacro (robot description, xacro)
@@ -2,7 +2,31 @@
 <robot xmlns:xacro="http://www.ros.org/wiki/xacro">
     <gazebo>
+        <!--plugin
+            filename="gz-sim-pose-publisher-system"
+            name="gz::sim::systems::PosePublisher">
+            <publish_link_pose>true</publish_link_pose>
+            <use_pose_vector_msg>true</use_pose_vector_msg>
+            <static_publisher>true</static_publisher>
+            <static_update_frequency>1</static_update_frequency>
+        </plugin-->
+        <!--plugin
+            filename="gz-sim-odometry-publisher-system"
+            name="gz::sim::systems::OdometryPublisher">
+            <odom_frame>robot/odom</odom_frame>
+            <robot_base_frame>robot/base_link</robot_base_frame>
+            <odom_publish_frequency>50</odom_publish_frequency>
+        </plugin-->
         <plugin
             filename="gz-sim-joint-state-publisher-system"
             name="gz::sim::systems::JointStatePublisher">
+        </plugin>
+        <plugin
+            filename="gz-sim-sensors-system"
+            name="gz::sim::systems::Sensors">
+        <render_engine>ogre2</render_engine>
+        </plugin>
+        <plugin
+            filename="gz-sim-imu-system"
+            name="gz::sim::systems::Imu">
         </plugin>
         <plugin
@@ -16,12 +40,4 @@
             <odom_publish_frequency>10</odom_publish_frequency>
         </plugin>
-        <plugin filename="gz-sim-imu-system"
-        	name="gz::sim::systems::Imu">
-	</plugin>
-	<plugin
-		filename="gz-sim-sensors-system"
-		name="gz::sim::systems::Sensors">
-	<render_engine>ogre2</render_engine>
-	</plugin>
     </gazebo>
 </robot>
